File: board_gw1/unic_gw1.kicad_sch (KiCad schematic)
At the start: 112 parts, among them Q1 2N7002, Q10 2N7002, Q11 2N7002, Q12 2N7002, Q13 2N7002, Q14 2N7002, Q15 2N7002, Q16 2N7002, Q17 2N7002, Q18 2N7002, Q19 2N7002, Q2 2N7002, Q20 2N7002, Q21 2N7002, Q22 2N7002, Q23 2N7002, Q24 2N7002, Q25 2N7002, Q26 2N7002, Q27 2N7002, Q28 2N7002, Q29 2N7002, Q3 2N7002, Q30 2N7002, Q31 2N7002, Q32 2N7002, Q33 2N7002, Q34 2N7002, Q35 2N7002, Q36 2N7002, Q37 2N7002, Q38 2N7002, Q39 2N7002, Q4 2N7002, Q40 2N7002, Q5 2N7002, Q6 2N7002, Q7 2N7002, Q8 2N7002, Q9 2N7002, U1 GW1N-LV9QN88C6_I5_, U2 LM3480-3.3, U3 AP2202K-ADJ, U4 APS6404L-3SQR-ZR, U6 AP62150Z6, U7 W25Q16JVUXIQ, X1 ASE-xxxMHz

Commit message: Reworked switcher components and layout.
Parts:
- C1, C11, C13, C14, C15, C16, C17, C18, C19, C2, C20, C21, C22, C23, C4, C6, C9: value 0.1u -> 2.2u; manf# (none) -> CC0402MRX5R6BB225
- C12: manf# (none) -> GRM188R61E106KA73J; now not fitted
- C3: manf# (none) -> CC0402MRX5R6BB225
- C5: footprint Capacitor_SMD:C_0805_2012Metric_Pad1.18x1.45mm_HandSolder -> Capacitor_SMD:C_0603_1608Metric_Pad1.08x0.95mm_HandSolder; manf# (none) -> GRM188R61E106KA73J
- C7: footprint Capacitor_SMD:C_0805_2012Metric_Pad1.18x1.45mm_HandSolder -> Capacitor_SMD:C_0603_1608Metric_Pad1.08x0.95mm_HandSolder; manf# (none) -> GRM188R60G226MEA0J
- C8: footprint Capacitor_SMD:C_0805_2012Metric_Pad1.18x1.45mm_HandSolder -> Capacitor_SMD:C_0603_1608Metric_Pad1.08x0.95mm_HandSolder; manf# (none) -> GRM188R60G226MEA0J; now not fitted
- D1, D11, D2, D3, D4, D5, D6, D7, D8, D9: manf# (none) -> BAT54DF
- D21, D22, D23, D24, D25, D26, D27, D28, D29, D30: manf# (none) -> BAT54CV\,115
- DISPLAY1: kicost:link (none) -> https://www.crystalfontz.com/product/cfal12832c0091bw-small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; kicost:pricing (none) -> 1:$6.59; 5:$5.51; 10:$5.36; 20:$5.18; 50:$5.00; 100:$4.92; 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; manf# (none) -> CFAL12832C-0091B-W_A
- J_DISPLAY1: manf# (none) -> FH19C-12S-0.5SH(10)
- J_EXT1: manf# (none) -> 502598-2793
- J_JTAG1: manf# (none) -> 10152265-1121HF; now not fitted
- L1: value 3.3uH -> 10uH; manf# (none) -> UHP 252012BF-100M
- LED_DONE1: manf# (none) -> CS42C-QL4
- Q1, Q10, Q11, Q12, Q13, Q14, Q15, Q16, Q17, Q18, Q19, Q2, Q20, Q21, Q22, Q23, Q24, Q25, Q26, Q27, Q28, Q29, Q3, Q30, Q31, Q32, Q33, Q34, Q35, Q36, Q37, Q38, Q39, Q4, Q40, Q5, Q6, Q7, Q8, Q9: manf# (none) -> 2N7002KL3A-TP
- R1: manf# (none) -> CR0402-JW-221GLF
- R10, R11, R12, R13, R15, R16, R3, R5, R6, R7, R8, R9: manf# (none) -> CR0402-FX-1002GLF
- R14, R4: manf# (none) -> ERJ-2RKF4991X
- R2: manf# (none) -> CR0402-JW-102GLF
- SOCKET1: manf# (none) -> BA3760-TUBL-4A-F5
- U1: kicost:pricing (none) -> 100:$5.80; 168:$5.41; 1000:$5.21; manf# (none) -> GW1N-LV9QN88C6/I5/
- U2: manf# (none) -> LM3480IM3X-3.3/NOPB
- U3: manf# (none) -> AP2202K-ADJTRE1
- U4: manf# (none) -> APS6404L-3SQR-ZR
- U6: manf# (none) -> AP62150Z6-7
- U7: manf# (none) -> W25Q16JVUXIQ TR
- X1: value ASE-xxxMHz -> 27MHz; manf# (none) -> O 27\,0-JO32-B-1V3-1-T1-LF
Other:
- note added: "Static input current for an LS gate is 0.1mA. This gives us <10mA static output current. We can sustain with an LDO See http://raven1.magix.net/Ti%20TTL%20DataBook%20vol1.pdf, page 20 https://ecelabs.njit.edu/fed101/resources/Motorola_Short_Version.pdf page 12 Detailed answer: https://electronics.stackexchange.com/questions/633886/what-does-limit-of-1-ttl-ls-load-mean"
- note removed: "Another option: Kyocera connector: https://ele.kyocera.com/assets/products/connector/6844.pdf Corresponding FPC cable: https://tools.molex.com/pdm_docs/sd/150320221_sd.pdf"
- note removed: "Molex connector: https://www.molex.com/en-us/products/part-detail/502598-2793 Mating cable: 15015-xx27 Corresponding flexes: https://rhu004.sma-promail.com/SQLImages/kelmscott/Molex/PDF_Images/987650-6721.PDF 0.3A per contact for the connector, 0.2A for the cable"
- note removed: "TODO: 3.3 needs to be a switcher! At 12V input power we can't sustain even 100mA I/O current. Static input current for an LS gate is 0.1mA. This gives us <10mA static output current. *THAT* We can sustain with an LDO See http://raven1.magix.net/Ti%20TTL%20DataBook%20vol1.pdf, page 20 https://ecelabs.njit.edu/fed101/resources/Motorola_Short_Version.pdf page 12 Detailed answer: https://electronics.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"
- note removed: "TODO: check pinout against uHDMI!"
- note removed: "TODO: make sure footprint matches TANG NANO 9k"
- note removed: "There are a ton of TVS diodes of this persuation: https://assets.nexperia.com/documents/data-sheet/IP4221CZ6-XS.pdf They are great, cheap, but can't stand more than 5V. They also have a 0.7V forward voltage. Another single-source solution: http://www.smc-diodes.com/propdf/BAT54DF%20N2313%20REV.-.pdf This is 4 pairs of diodes in one package. Not replacing as current option with several second sour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"
- note removed: "There are dual- 7002 devices. https://assets.nexperia.com/documents/data-sheet/NX7002BKXB.pdf https://toshiba.semicon-storage.com/info/SSM6N7002BFE_datasheet_en_20140301.pdf?did=2282&prodName=SSM6N7002BFE https://www.diodes.com/assets/Datasheets/ds30639.pdf - has multiple sources Single ones: NX7002BKH or NX7002BKM"
- note removed: "Trion (T8Q144C3) FPGAs are *much* cheaper, but they have package issues: BGA81 is the closest to something that would work The T13F169C3 thingy is in 169-pin BGA (can be escaped on two layers, but need via-in-pad) for $7"

Commit message: Switched back to 0805 caps: they're cheaper. TODO: part number updates.
Parts:
- C12, C5, C7, C8: footprint Capacitor_SMD:C_0603_1608Metric_Pad1.08x0.95mm_HandSolder -> Capacitor_SMD:C_0805_2012Metric_Pad1.18x1.45mm_HandSolder
Changed lines of the file:
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@@
       (effects (font (size 1.27 1.27)) (justify left))
     )
-    (property "Footprint" "Capacitor_SMD:C_0603_1608Metric_Pad1.08x0.95mm_HandSolder" (at 227.33 48.26 0)
+    (property "Footprint" "Capacitor_SMD:C_0805_2012Metric_Pad1.18x1.45mm_HandSolder" (at 227.33 48.26 0)
       (effects (font (size 1.27 1.27)) hide)
     )
@@
       (effects (font (size 1.27 1.27)) (justify left))
     )
-    (property "Footprint" "Capacitor_SMD:C_0603_1608Metric_Pad1.08x0.95mm_HandSolder" (at 238.76 266.7 0)
+    (property "Footprint" "Capacitor_SMD:C_0805_2012Metric_Pad1.18x1.45mm_HandSolder" (at 238.76 266.7 0)
       (effects (font (size 1.27 1.27)) hide)
     )
@@
       (effects (font (size 1.27 1.27)) (justify left))
     )
-    (property "Footprint" "Capacitor_SMD:C_0603_1608Metric_Pad1.08x0.95mm_HandSolder" (at 185.42 266.7 0)
+    (property "Footprint" "Capacitor_SMD:C_0805_2012Metric_Pad1.18x1.45mm_HandSolder" (at 185.42 266.7 0)
       (effects (font (size 1.27 1.27)) hide)
     )
@@
       (effects (font (size 1.27 1.27)) (justify left))
     )
-    (property "Footprint" "Capacitor_SMD:C_0603_1608Metric_Pad1.08x0.95mm_HandSolder" (at 242.57 266.7 0)
+    (property "Footprint" "Capacitor_SMD:C_0805_2012Metric_Pad1.18x1.45mm_HandSolder" (at 242.57 266.7 0)
       (effects (font (size 1.27 1.27)) hide)
     )

Commit message: Ready to roll with DEVEL board!
Parts:
- C12, C5: manf# GRM188R61E106KA73J -> CL21A106KAYNNNG
- C7, C8: manf# GRM188R60G226MEA0J -> CL21A226MQQNNNE
- J_DISPLAY1: footprint UNIC:HRS_FH19C-12S-0.5SH_05_ -> UNIC:CF31121D0R0-05-NH; manf# FH19C-12S-0.5SH(10) -> CF31121D0R0-05-NH
Connections:
- net +3V3: now also J_DISPLAY1.2 (Pin_2), J_DISPLAY1.3 (Pin_3), J_DISPLAY1.4 (Pin_4); no longer J_DISPLAY1.10 (Pin_10), J_DISPLAY1.11 (Pin_11), J_DISPLAY1.9 (Pin_9)
- net GND: now also J_DISPLAY1.5 (Pin_5); no longer J_DISPLAY1.8 (Pin_8)
- net LCD_CS_N: now also J_DISPLAY1.6 (Pin_6); no longer J_DISPLAY1.7 (Pin_7)
- net LCD_RST_N: now also J_DISPLAY1.7 (Pin_7); no longer J_DISPLAY1.6 (Pin_6)
- net SPI_CLK: now also J_DISPLAY1.9 (Pin_9); no longer J_DISPLAY1.4 (Pin_4)
- net SPI_MOSI_IO0: now also J_DISPLAY1.10 (Pin_10); no longer J_DISPLAY1.3 (Pin_3)
Other:
- note added: "BS0"
- note added: "BS1"
- note added: "CS#"
- note added: "D/C#"
- note added: "D0"
- note added: "D1"
- note added: "D2"
- note added: "GND"
- note added: "Pinout is reversed compared to datasheet due to use of bottom-contact connector"
- note added: "RES#"
- note added: "VBAT"
- note added: "VDD"
- note added: "Volume PCB Assembly BOM Total ======== ======= ========= ======= ======= 100 1.5 4.3 22.05 27.85 200 1.08 2.8 21.61 25.49 1000 0.43 1.3 19.49 21.22"
- note removed: "PCB cost seems to be $350 for setup including 4 layers and via-in-pad. That gives us about 100 boards for the same price (i.e. unit-cost is $0). For 1000 boards, we get $650 cost. Without via-in-pad, it seems we can have a 100 boards for $160 Assembly for the same seems to be around $400 for 100 pieces. So, total 'transformation cost' appears to be around $5, if I can get an order of a 100 togeth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"
- moved on the sheet: C11
