File: devel_gw1/devel_gw1.kicad_sch (KiCad schematic)
At the start: 180 parts, among them J2 Conn_01x02, Q1 2N7002, Q10 2N7002, Q11 2N7002, Q12 2N7002, Q13 2N7002, Q14 2N7002, Q15 2N7002, Q16 2N7002, Q17 2N7002, Q18 2N7002, Q19 2N7002, Q2 2N7002, Q20 2N7002, Q21 2N7002, Q22 2N7002, Q23 2N7002, Q24 2N7002, Q25 2N7002, Q26 2N7002, Q27 2N7002, Q28 2N7002, Q29 2N7002, Q3 2N7002, Q30 2N7002, Q31 2N7002, Q32 2N7002, Q33 2N7002, Q34 2N7002, Q35 2N7002, Q36 2N7002, Q37 2N7002, Q38 2N7002, Q39 2N7002, Q4 2N7002, Q41 2N7002, Q5 2N7002, Q6 2N7002, Q7 2N7002, Q8 2N7002, Q9 2N7002, U1 GW1N-LV9QN88C6_I5_, U2 LM3480-3.3, U3 AP2202K-ADJ, U4 APS6404L-3SQR-SN, U6 AP62150Z6, U7 AT25SF081-SSHB-X, X1 27MHz

Commit message: Ready to roll with DEVEL board!
Parts:
- added J_DISPLAY3: Conn_01x12_MountingPin, UNIC:CF31121D0R0-05-NH, symbol Connector_Generic_MountingPin:Conn_01x12_MountingPin
- C1, C10, C11, C13, C14, C15, C16, C17, C18, C19, C2, C20, C21, C22, C23, C4, C6, C9: value 0.1u -> 2.2u; manf# (none) -> CC0402MRX5R6BB225
- C12: footprint Capacitor_SMD:C_0603_1608Metric_Pad1.08x0.95mm_HandSolder -> Capacitor_SMD:C_0805_2012Metric_Pad1.18x1.45mm_HandSolder; manf# (none) -> CL21A106KAYNNNG; now not fitted
- C3: manf# (none) -> CC0402MRX5R6BB225
- C5: manf# (none) -> CL21A106KAYNNNG
- C7: manf# (none) -> CL21A226MQQNNNE
- C8: manf# (none) -> CL21A226MQQNNNE; now not fitted
- D1, D11, D13, D15, D17, D19, D2, D21, D23, D25, D27, D29, D31, D33, D35, D37, D39, D4, D41, D43, D45, D47, D49, D51, D53, D55, D57, D59, D6, D61, D63, D65, D67, D69, D71, D73, D75, D77, D79, D8: MP BAT54-7-F -> (none); manf# (none) -> BAT54-7-F
- D10, D12, D14, D16, D18, D20, D22, D24, D26, D28, D3, D30, D32, D34, D36, D38, D40, D42, D44, D46, D48, D5, D50, D52, D54, D56, D58, D60, D62, D64, D66, D68, D7, D70, D72, D74, D76, D78, D80, D9: MP BAT54S-7-F -> (none); manf# (none) -> BAT54S-7-F
- DISPLAY1: kicost:link (none) -> https://www.crystalfontz.com/product/cfal12832c0091bw-small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; kicost:pricing (none) -> 1:$6.59; 5:$5.51; 10:$5.36; 20:$5.18; 50:$5.00; 100:$4.92; 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; now fitted
- J2, JP1, JP2, JP3, JP4: MP PRPC002SAAN-RC -> (none); manf# (none) -> PRPC002SAAN-RC
- J_DISPLAY1: footprint UNIC:HRS_FH19C-12S-0.5SH_05_ -> UNIC:CF4212FH0R0-05-NH; MP FH19C-12S-0.5SH(10) -> (none); manf# (none) -> CF4212FH0R0-05-NH
- J_DISPLAY2: MP PRPC012SAAN-RC -> (none); manf# (none) -> PRPC012SAAN-RC
- J_EXT1: MP 502598-2793 -> (none); manf# (none) -> 502598-2793
- J_EXT2: MP PRPC014DAAN-RC -> (none); manf# (none) -> PRPC014DAAN-RC
- J_JTAG1: MP 10152265-1121HF -> (none); kicost:link (none) -> https://www.crystalfontz.com/product/cfal12832c0091bw-small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; kicost:pricing (none) -> 1:$6.59; 5:$5.51; 10:$5.36; 20:$5.18; 50:$5.00; 100:$4.92; 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; manf# (none) -> 10152265-1121HF
- L1: value 3.3uH -> 10uH; MP WIP252012S-3R3MLDG -> (none); manf# (none) -> UHP 252012BF-100M
- LED_DONE1: MP CS42C-QL4 -> (none); manf# (none) -> CS42C-QL4
- Q1, Q10, Q11, Q12, Q13, Q14, Q15, Q16, Q17, Q18, Q19, Q2, Q20, Q21, Q22, Q23, Q24, Q25, Q26, Q27, Q28, Q29, Q3, Q30, Q31, Q32, Q33, Q34, Q35, Q36, Q37, Q38, Q39, Q4, Q41, Q5, Q6, Q7, Q8, Q9: MP NDS7002A -> (none); manf# (none) -> 2N7002NXAKR
- R1: manf# (none) -> CR0402-JW-221GLF
- R10, R11, R12, R13, R15, R16, R3, R5, R6, R7, R8, R9: manf# (none) -> CR0402-FX-1002GLF
- R14, R4: manf# (none) -> ERJ-2RKF4991X
- R2: manf# (none) -> CR0402-JW-102GLF
- SOCKET1: manf# (none) -> PPPC202LJBN-RC
- U1: MP GW1N-LV9QN88C6/I5/ -> (none); kicost:pricing (none) -> 100:$5.80; 168:$5.41; 1000:$5.21; manf# (none) -> GW1N-LV9QN88C6/I5/
- U2: MP LM3480IM3X-3.3/NOPB -> (none); manf# (none) -> LM3480IM3X-3.3/NOPB
- U3: MP AP2202K-ADJTRE1 -> (none); manf# (none) -> AP2202K-ADJTRE1
- U4: MP APS6404L-3SQR-SN -> (none); manf# (none) -> APS6404L-3SQR-SN
- U6: MP AP62150Z6-7 -> (none); manf# (none) -> AP62150Z6-7
- U7: MP AT25SF081B-SSHB-T -> (none); manf# (none) -> AT25SF081B-SSHB-T
- X1: MP O 27\,0-JO32-B-1V3-1-T1-LF -> (none); manf# (none) -> O 27\,0-JO32-B-1V3-1-T1-LF
Connections:
- net +3V3: now also J_DISPLAY3.2 (Pin_2), J_DISPLAY3.3 (Pin_3), J_DISPLAY3.4 (Pin_4)
- net GND: now also J_DISPLAY3.1 (Pin_1), J_DISPLAY3.12 (Pin_12), J_DISPLAY3.5 (Pin_5), J_DISPLAY3.MP (MountPin)
- net LCD_CS_N: now also J_DISPLAY3.6 (Pin_6)
- net LCD_RST_N: now also J_DISPLAY3.7 (Pin_7)
- net SPI_CLK: now also J_DISPLAY3.9 (Pin_9)
- net SPI_MOSI_IO0: now also J_DISPLAY3.10 (Pin_10)
- no-connect marks 5 -> 7
Other:
- note added: "BS0"
- note added: "BS1"
- note added: "Below 100mA (maybe even as low as 300mA) the switcher operaters in PFM mode with this inductor setting. A heavily utilized FPGA would on the order of 200mA. So, maybe a larger inductor is called for?"
- note added: "CS#"
- note added: "D/C#"
- note added: "D0"
- note added: "D1"
- note added: "D2"
- note added: "GND"
- note added: "Pinout is reversed compared to datasheet due to use of bottom-contact connector"
- note added: "RES#"
- note added: "Static input current for an LS gate is 0.1mA. This gives us <10mA static output current. We can sustain with an LDO See http://raven1.magix.net/Ti%20TTL%20DataBook%20vol1.pdf, page 20 https://ecelabs.njit.edu/fed101/resources/Motorola_Short_Version.pdf page 12 Detailed answer: https://electronics.stackexchange.com/questions/633886/what-does-limit-of-1-ttl-ls-load-mean"
- note added: "VBAT"
- note added: "VDD"
- note removed: "Another option: Kyocera connector: https://ele.kyocera.com/assets/products/connector/6844.pdf Corresponding FPC cable: https://tools.molex.com/pdm_docs/sd/150320221_sd.pdf"
- note removed: "Molex connector: https://www.molex.com/en-us/products/part-detail/502598-2793 Mating cable: 15015-xx27 Corresponding flexes: https://rhu004.sma-promail.com/SQLImages/kelmscott/Molex/PDF_Images/987650-6721.PDF 0.3A per contact for the connector, 0.2A for the cable"
- note removed: "Probably want the APS6404L-3SQR-SN variant: $1.46 @ Mouser"
- note removed: "TODO: 3.3 needs to be a switcher! At 12V input power we can't sustain even 100mA I/O current. Static input current for an LS gate is 0.1mA. This gives us <10mA static output current. *THAT* We can sustain with an LDO See http://raven1.magix.net/Ti%20TTL%20DataBook%20vol1.pdf, page 20 https://ecelabs.njit.edu/fed101/resources/Motorola_Short_Version.pdf page 12 Detailed answer: https://electronics.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"
- note removed: "TODO: check pinout against uHDMI!"
- note removed: "TODO: make sure footprint matches TANG NANO 9k"
- note removed: "There are a ton of TVS diodes of this persuation: https://assets.nexperia.com/documents/data-sheet/IP4221CZ6-XS.pdf They are great, cheap, but can't stand more than 5V. They also have a 0.7V forward voltage. Another single-source solution: http://www.smc-diodes.com/propdf/BAT54DF%20N2313%20REV.-.pdf This is 4 pairs of diodes in one package. Not replacing as current option with several second sour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"
- note removed: "There are dual- 7002 devices. https://assets.nexperia.com/documents/data-sheet/NX7002BKXB.pdf https://toshiba.semicon-storage.com/info/SSM6N7002BFE_datasheet_en_20140301.pdf?did=2282&prodName=SSM6N7002BFE https://www.diodes.com/assets/Datasheets/ds30639.pdf - has multiple sources Single ones: NX7002BKH or NX7002BKM"
- note removed: "Trion (T8Q144C3) FPGAs are *much* cheaper, but they have package issues: BGA81 is the closest to something that would work The T13F169C3 thingy is in 169-pin BGA (can be escaped on two layers, but need via-in-pad) for $7"
- moved on the sheet: C11, SOCKET1

Commit message: Devel updates.
Parts:
- LED_DONE1: manf# CS42C-QL4 -> B1811NG--05D001013U1930
- R14: value 4.99k -> 29.4k; manf# ERJ-2RKF4991X -> (none)
Other:
- note added: "5V is trimmed to 4.88V"
- note removed: "5V is trimmed to 4.5V"
Changed lines of the file:
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@@
     (effects (font (size 1.27 1.27)) (justify left bottom))
   )
-  (text "5V is trimmed to 4.5V" (at 176.53 273.05 0)
+  (text "5V is trimmed to 4.88V" (at 176.53 273.05 0)
     (effects (font (size 1.27 1.27)) (justify left bottom))
   )
@@
   (symbol (lib_id "Device:R_Small_US") (at 163.83 287.02 0) (unit 1)
     (in_bom yes) (on_board yes) (dnp no) (fields_autoplaced)
-    (property "Reference" "R14" (at 166.37 285.7499 0)
+    (property "Reference" "R14" (at 166.37 285.75 0)
       (effects (font (size 1.27 1.27)) (justify left))
     )
-    (property "Value" "4.99k" (at 166.37 288.2899 0)
+    (property "Value" "29.4k" (at 166.37 288.29 0)
       (effects (font (size 1.27 1.27)) (justify left))
     )
@@
       (effects (font (size 1.27 1.27)) hide)
     )
-    (property "manf#" "ERJ-2RKF4991X" (at 163.83 287.02 0)
+    (property "manf#" "" (at 163.83 287.02 0)
       (effects (font (size 1.27 1.27)) hide)
     )
@@
       (effects (font (size 1.27 1.27)) hide)
     )
-    (property "Datasheet" "https://chromeled.com/pdf/smd/CS42C-QL4.pdf" (at 67.31 100.33 0)
+    (property "Datasheet" "https://mm.digikey.com/Volume0/opasdata/d220001/medias/docus/3815/B1811NG--05D001013U1930.pdf" (at 67.31 100.33 0)
       (effects (font (size 1.27 1.27)) hide)
     )
-    (property "manf#" "CS42C-QL4" (at 67.31 100.33 90)
+    (property "manf#" "B1811NG--05D001013U1930" (at 67.31 100.33 90)
       (effects (font (size 1.27 1.27)) hide)
     )
