File: programmer/programmer.kicad_pcb (KiCad board)
At the start: 2 copper layers, 63 x 30 mm, 50 parts, among them J1 USB_C_Receptacle_USB2.0_14P, U1 FT2232HL, U2 74LVC2T45DC, U3 93CxxA, U4 NLSV2T244DM, U5 NLSV2T244DM, U6 NLSV2T244DM, U8 AMS1117-3.3, Y1 12MHz

Commit message: Release package for programmer.
Parts:
- added D4: LED, LED_SMD:LED_0603_1608Metric_Pad1.05x0.95mm_HandSolder, F.Cu at (52.0, 22.6)
- added D5: LED, LED_SMD:LED_0603_1608Metric_Pad1.05x0.95mm_HandSolder, F.Cu at (50.2, 22.6)
- added R10: 220, Resistor_SMD:R_0603_1608Metric_Pad0.98x0.95mm_HandSolder, F.Cu at (52.0, 26.1)
- added R11: 220, Resistor_SMD:R_0603_1608Metric_Pad0.98x0.95mm_HandSolder, F.Cu at (50.2, 26.1)
- moved D3 4.80 mm to (52.6, 30.7)
- moved C2 2.71 mm to (89.0, 36.7)
- moved C9 2.56 mm to (67.1, 23.5), turned to 90 degrees
- moved U2 1.86 mm to (63.8, 23.9)
- moved R4 1.60 mm to (99.2, 28.7)
- moved R9 1.44 mm to (91.6, 37.3), turned to -90 degrees
- moved R8 0.82 mm to (93.4, 42.7)
- moved C18 0.60 mm to (65.3, 29.7)
- moved R7 0.52 mm to (93.4, 44.6)
- moved D1 0.45 mm to (90.5, 33.6)
- moved R6 0.33 mm to (93.4, 46.4)
- moved J1 0.30 mm to (99.0, 35.0)
Connections:
- net Net-(J1-SHIELD) renamed /SHIELD
Routing:
- net VIO: track 81.0 -> 12.4 mm, vias 6 -> 7
- net VCC: track 137.8 -> 74.0 mm, vias 16 -> 15
- net /FT_JTAG_EN_N: track 33.9 -> 56.3 mm, vias 0 -> 4
- net /JTAG_TDI: track 59.9 -> 55.4 mm, vias 0 -> 2
- net Net-(JP3-A): track 3.75 -> 8.08 mm
- net /JTAG_TMS: track 53.6 -> 56.2 mm
- net GND: track 50.0 -> 52.3 mm
- net Net-(U1-REF): track 8.10 -> 10.4 mm
- net Net-(D5-A): track 0.00 -> 1.71 mm
- net Net-(D4-A): track 0.00 -> 1.71 mm
- net Net-(U1-VPHY): track 4.91 -> 6.53 mm
- net /FT_JTAG_TDO: track 19.8 -> 21.3 mm
- net +5V: track 26.5 -> 25.0 mm, vias 2 -> 0
- net /SHIELD: track 19.8 -> 19.0 mm
- net Net-(JP1-A): track 6.28 -> 7.03 mm
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- added copper zone on F.Cu, net /SHIELD
- added copper zone on F.Cu, net VCC
- added copper zone on F.Cu, net VIO
Other:
- board text added: "JTAG_SEL"
- board text added: "RECONFIG"
- board text added: "SER_RXD"
- board text added: "SER_TXD"
- board text added: "TARGET"
- board text added: "USB"
