File: programmer/programmer.kicad_sch (KiCad schematic)
At the start: 50 parts, among them J1 USB_C_Receptacle_USB2.0_14P, U1 FT2232HL, U2 74LVC2T45DC, U3 93CxxA, U4 NLSV2T244DM, U5 NLSV2T244DM, U6 NLSV2T244DM, U8 AMS1117-3.3, Y1 12MHz

Commit message: Release package for programmer.
Parts:
- added D4, D5: LED, LED_SMD:LED_0603_1608Metric_Pad1.05x0.95mm_HandSolder, symbol Device:LED
- added R10, R11: 220, Resistor_SMD:R_0603_1608Metric_Pad0.98x0.95mm_HandSolder, symbol Device:R_Small_US
- J1: mpn (none) -> 44116B01231
Connections:
- net FT_JTAG_EN_N: now also R10.2
- net GND: now also R11.2
- net VCC: now also D4.1 (K)
- net VIO: now also D5.1 (K)
- net SHIELD: now reaches J1.S1 (SHIELD), R4.1
- new net: D5.2 (A), R11.1
- new net: D4.2 (A), R10.1
Other:
- moved on the sheet: R4

Commit message: Added BOM notes
Parts:
- C1, C10, C11, C12, C13, C14, C15, C16, C17, C18, C19, C2, C3, C4, C5, C6, C7, C8, C9, D4, D5, H1, H2, H3, H4, JP1, JP2, JP3, JP4, J_EXT2, R1, R10, R11, R2, R3, R4, R5, R6, R7, R8, R9, U1, U3, U8, Y1: HAVE IT (none) -> YES

Commit message: Programmer bring-up changes and notes
Parts:
- added C20, C21, C22: 3.3u, Capacitor_SMD:C_0603_1608Metric_Pad1.08x0.95mm_HandSolder, symbol Device:C_Small
- added R12: 2.2, Resistor_SMD:R_0603_1608Metric_Pad0.98x0.95mm_HandSolder, symbol Device:R_Small_US
- added TP1, TP2, TP3, TP4, TP5, TP6: TestPoint, TestPoint:TestPoint_THTPad_1.0x1.0mm_Drill0.5mm, symbol Connector:TestPoint
- C6: value 3.3u -> 22u; footprint Capacitor_SMD:C_0603_1608Metric_Pad1.08x0.95mm_HandSolder -> Capacitor_SMD:C_0805_2012Metric_Pad1.18x1.45mm_HandSolder
- J1: mpn 44116B01231 -> USB4215-03-A
Connections:
- net GND: now also C20.2, C21.2, C22.2, R12.2; no longer C6.2
- net VCC: now also D4.2 (A); no longer D4.1 (K)
- net VIO: now also D5.2 (A), C20.1, C21.1, C22.1; no longer D5.1 (K)
- net at R11.1: now also D5.1 (K); no longer D5.2 (A)
- net at U1.32 (ACBUS5): now also TP1.1
- net at U1.33 (ACBUS6): now also TP2.1
- net at U1.34 (ACBUS7): now also TP3.1
- net at U1.45 (BDBUS6): now also TP6.1
- net at U1.46 (BDBUS7): now also TP5.1
- net at U1.48 (BCBUS0): now also TP4.1
- net at R10.1: now also D4.1 (K); no longer D4.2 (A)
- new net: C6.2, R12.1
Other:
- note added: "ADDED PULL-UP ON TDO. NOT SURE IF NEEDED"
- note added: "REALLY NEED TO FIND A BETTER LDO"
- note added: "THIS ESD DIODE DOESN'T WORK FOR USB AT LEAST!"
- moved on the sheet: D4, D5

Commit message: Updated programmer schematic and PCBs.
All known changes are incorporated.

p.s.: I decided to stick with this rather sketchy LDO.
The reason for this is that it's heatsink tab is connected
to VCC, which happens to be the fill on the top layer
so a GND-connected alternative would be less well cooled.
Parts:
- added R13: 10k, Resistor_SMD:R_0603_1608Metric_Pad0.98x0.95mm_HandSolder, symbol Device:R_Small_US
- D1, D2, D3: now not fitted
Connections:
- net JTAG_TDO: now also R13.2
- net VIO: now also R13.1
Other:
- note removed: "ADDED PULL-UP ON TDO. NOT SURE IF NEEDED"
- note removed: "REALLY NEED TO FIND A BETTER LDO"
- title: UNIC 40 -> UNIC Programmer
- moved on the sheet: C1, C10, C11, C12, C13, C14, C15, C16, C17, C18, C19, C2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
