File: shadow_tracer/shadow_tracer.kicad_pcb (KiCad board)
At the start: 2 copper layers, 55.9 x 111.8 mm, 8 parts, among them J1 Conn_01x08, J2 Conn_01x20, J3 Conn_01x20

Commit message: Shadow tracer release package.
Parts:
- added J4: Conn_01x08, Connector_PinHeader_2.54mm:PinHeader_1x02_P2.54mm_Vertical, F.Cu at (174.8, 158.2)
- added J5: Conn_01x08, Connector_PinHeader_2.54mm:PinHeader_1x02_P2.54mm_Vertical, F.Cu at (125.2, 84.6)
- added J6: Conn_01x08, Connector_PinHeader_2.54mm:PinHeader_1x02_P2.54mm_Vertical, F.Cu at (124.0, 158.2)
- added J7: Conn_01x08, Connector_PinHeader_2.54mm:PinHeader_1x02_P2.54mm_Vertical, F.Cu at (154.0, 71.9)
- added J8: Conn_01x08, Connector_PinHeader_2.54mm:PinHeader_1x02_P2.54mm_Vertical, F.Cu at (158.7, 71.9)
- added J9: Conn_01x08, Connector_PinHeader_2.54mm:PinHeader_1x02_P2.54mm_Vertical, F.Cu at (163.3, 71.9)
- moved J1 2.83 mm to (173.5, 85.9)
Connections:
- J_EXT1 pad MP: GND -> GNDI
Routing:
- net /PIN21: track 73.6 -> 74.6 mm
- net /FPC25: track 25.3 -> 26.1 mm
- net /FPC18: track 14.6 -> 14.0 mm
- added copper zone on B.Cu, net GND
- added copper zone on F.Cu, net GNDI
- removed copper zone on F.Cu, net GND
Other:
- board text added: "1"
- board text added: "10"
- board text added: "15"
- board text added: "20"
- board text added: "21"
- board text added: "25"
- board text added: "30"
- board text added: "35"
- board text added: "40"
- board text added: "5"
