File: shadow_tracer/shadow_tracer.kicad_sch (KiCad schematic)
At the start: 8 parts, among them J1 Conn_01x08, J2 Conn_01x20, J3 Conn_01x20

Commit message: Shadow tracer release package.
Parts:
- added J4, J5, J6, J7, J8, J9: Conn_01x08, Connector_PinHeader_2.54mm:PinHeader_1x02_P2.54mm_Vertical, symbol Connector_Generic:Conn_01x02
Connections:
- net GND: now also J4.1 (Pin_1), J4.2 (Pin_2), J5.1 (Pin_1), J5.2 (Pin_2), J6.1 (Pin_1), J6.2 (Pin_2); no longer J_EXT1.MP (MountPin)
- new net GNDI: J7.1 (Pin_1), J7.2 (Pin_2), J8.1 (Pin_1), J8.2 (Pin_2), J9.1 (Pin_1), J9.2 (Pin_2), J_EXT1.MP (MountPin)

Commit message: Some quick schematic beautification.
Other:
- title: UNIC 40 -> UNIC 40 Shadow Tracer
Changed lines of the file:
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@@
 	(paper "A")
 	(title_block
-		(title "UNIC 40")
-		(date "2023-11-24")
+		(title "UNIC 40 Shadow Tracer")
+		(date "2024-09-01")
 		(rev "1.0")
 		(company "Modular Circuits")
@@
 		(dnp no)
 		(property "Reference" "J3"
-			(at 238.76 139.6999 0)
+			(at 242.062 111.76 0)
 			(effects
 				(font
@@
 		)
 		(property "Value" "Conn_01x20"
-			(at 238.76 142.2399 0)
+			(at 250.444 114.046 0)
 			(effects
 				(font
@@
 		(on_board yes)
 		(dnp no)
-		(fields_autoplaced yes)
 		(property "Reference" "J2"
-			(at 233.68 139.6999 0)
+			(at 229.616 111.76 0)
 			(effects
 				(font
@@
 		)
 		(property "Value" "Conn_01x20"
-			(at 233.68 142.2399 0)
+			(at 225.044 114.046 0)
 			(effects
 				(font
