File: z80_sampler/z80_sampler.kicad_sch (KiCad schematic)
At the start: 21 parts, among them U2 74HCT574, U3 74HCT10, U4 74HC86, U6 74HCT574, U7 74HCT245

Commit message: Z80 sampler project complete.
Parts:
- added C7: 1u, Capacitor_SMD:C_0603_1608Metric_Pad1.08x0.95mm_HandSolder, symbol Device:C_Small
- added JP4, JP6, JP7, JP8: Jumper_2_Bridged, Connector_PinHeader_2.54mm:PinHeader_1x02_P2.54mm_Vertical, symbol Jumper:Jumper_2_Bridged
- added JP5: Jumper_2_Open, Connector_PinHeader_2.54mm:PinHeader_1x02_P2.54mm_Vertical, symbol Jumper:Jumper_2_Open
- added JP9: Jumper_3_Bridged12, Connector_PinHeader_2.54mm:PinHeader_1x03_P2.54mm_Vertical, symbol Jumper:Jumper_3_Bridged12
- added R5, R6, R7, R8, R9: 10k, Resistor_SMD:R_0603_1608Metric_Pad0.98x0.95mm_HandSolder, symbol Device:R_Small_US
- added TP1: TestPoint, Connector_PinHeader_2.54mm:PinHeader_1x01_P2.54mm_Vertical, symbol Connector:TestPoint
- added U1: 74AHCT1G08, Package_TO_SOT_SMD:SOT-353_SC-70-5_Handsoldering, symbol 74xGxx:74AHCT1G08
- C1, C2, C3, C4, C5, C6: footprint Capacitor_THT:C_Disc_D4.3mm_W1.9mm_P5.00mm -> Capacitor_SMD:C_0603_1608Metric_Pad1.08x0.95mm_HandSolder
- R1, R2, R3, R4: footprint Resistor_THT:R_Axial_DIN0204_L3.6mm_D1.6mm_P5.08mm_Horizontal -> Resistor_SMD:R_0603_1608Metric_Pad0.98x0.95mm_HandSolder
- RV1: footprint Potentiometer_THT:Potentiometer_Runtron_RM-065_Vertical -> Potentiometer_Bourns_TC33X_Vertical; mpn (none) -> TC33X-2-101E
- U2, U6: footprint Package_DIP:DIP-20_W7.62mm_LongPads -> Package_SO:SOIC-20W_7.5x12.8mm_P1.27mm
- U3, U4: footprint Package_DIP:DIP-14_W7.62mm_LongPads -> Package_SO:SOIC-14_3.9x8.7mm_P1.27mm
- U7: value 74HCT245 -> SN74CBT3245CDW; footprint Package_DIP:DIP-20_W7.62mm_LongPads -> Package_SO:SOIC-20W_7.5x12.8mm_P1.27mm
Connections:
- net BUSREQ_N: now also U2.18 (Q1); no longer U2.17 (Q2)
- net CLK: now also TP1.1
- net CLK_2X: now also JP6.1 (A), JP9.3 (B); no longer U6.11 (Cp)
- net CLK_N: now also JP9.1 (A); no longer U2.11 (Cp)
- net D0: now also U7.8 (A6); no longer U7.12 (B6)
- net D1: now also U7.9 (A7); no longer U7.11 (B7)
- net D2: now also U7.6 (A4); no longer U7.14 (B4)
- net D3: now also U7.3 (A1); no longer U7.17 (B1)
- net D4: now also U7.2 (A0); no longer U7.18 (B0)
- net D5: now also U7.4 (A2); no longer U7.16 (B2)
- net D6: now also U7.5 (A3); no longer U7.15 (B3)
- net D7: now also U7.7 (A5); no longer U7.13 (B5)
- net GND: now also C7.2, R7.2, R9.2, U1.3 (GND); no longer U7.1 (A->B)
- net HOST_BUSREQ_N: now also U2.3 (D1); no longer U2.4 (D2)
- net HOST_D0: now also U7.12 (B6); no longer U7.8 (A6)
- net HOST_D1: now also U7.11 (B7); no longer U7.9 (A7)
- net HOST_D2: now also U7.14 (B4); no longer U7.6 (A4)
- net HOST_D3: now also U7.17 (B1); no longer U7.3 (A1)
- net HOST_D4: now also U7.18 (B0); no longer U7.2 (A0)
- net HOST_D5: now also U7.16 (B2); no longer U7.4 (A2)
- net HOST_D6: now also U7.15 (B3); no longer U7.5 (A3)
- net HOST_D7: now also U7.13 (B5); no longer U7.7 (A5)
- net HOST_INT_N: now also U2.2 (D0); no longer U2.3 (D1)
- net HOST_NMI_N: now also U2.4 (D2); no longer U2.2 (D0)
- net HOST_WAIT_N: now also JP2.3 (B), U1.2; no longer JP2.1 (A)
- net INT_N: now also U2.19 (Q0); no longer U2.18 (Q1)
- net NMI_N: now also U2.17 (Q2); no longer U2.19 (Q0)
- net RD_N: now also U4.13, JP4.1 (A), JP5.1 (A)
- net VCC: now also C7.1, R5.1, R6.1, R8.1, U1.5 (VCC)
- net at U2.15 (Q4): now also U1.1; no longer JP2.3 (B)
- net at U3.6: now also JP8.1 (A); no longer U7.19 (CE)
- net at U6.1 (OE): now also JP7.2 (B), R8.2; no longer U3.8
- net RN_N: no longer names the net of U3.5
- net RN_N: now also JP4.2 (B), R5.2; no longer U4.13
- new net: JP8.2 (B), R9.1, U7.19 (CE)
- new net: JP2.1 (A), U1.4
- new net: JP5.2 (B), R6.2, U7.1 (A->B)
- new net: JP9.2 (C), R7.1, U2.11 (Cp)
- new net: JP7.1 (A), U3.8
- new net: JP6.2 (B), U6.11 (Cp)
Other:
- note added: "Good selection guide for bus isolators: https://www.ti.com/lit/ml/scdb006a/scdb006a.pdf"
- moved on the sheet: C1, C2, C3, C4, C5, C6, CONN2, JP1, JP2, R1, RV1, U3C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

Commit message: Some small outstanding changes.
Parts:
- C1: mpn (none) -> C0603C102K5RACTU
- C2, C3, C4, C5, C6, C7: mpn (none) -> CL10B105KP8NNNC
- CONN1: mpn (none) -> PPPC202LJBN-RC
- CONN2: mpn (none) -> PH2RA-40-UA
- R1, R2, R3, R4, R5, R6, R7, R8, R9: mpn (none) -> RMCF0603JT10K0
- U1: mpn (none) -> 74AHCT1G08GW,125
- U2, U6: mpn (none) -> SN74HCT574DWR
- U3: mpn (none) -> 74HCT10D,653
- U4: value 74HC86 -> 74HCT86; mpn (none) -> 74HCT86D,653
- U7: mpn (none) -> SN74CBT3245CDW
