File: board_gw1_usb/board_gw1_usb.kicad_sch (KiCad schematic)
At the start: 203 parts, among them J1 USB_C_Receptacle, Q1 2N7002, Q10 2N7002, Q11 2N7002, Q12 2N7002, Q13 2N7002, Q14 2N7002, Q15 2N7002, Q16 2N7002, Q17 2N7002, Q18 2N7002, Q19 2N7002, Q2 2N7002, Q20 2N7002, Q21 2N7002, Q22 2N7002, Q23 2N7002, Q24 2N7002, Q25 2N7002, Q26 2N7002, Q27 2N7002, Q28 2N7002, Q29 2N7002, Q3 2N7002, Q30 2N7002, Q31 2N7002, Q32 2N7002, Q33 2N7002, Q34 2N7002, Q35 2N7002, Q36 2N7002, Q37 2N7002, Q38 2N7002, Q39 2N7002, Q4 2N7002, Q40 2N7002, Q41 2N7002, Q5 2N7002, Q6 2N7002, Q7 2N7002, Q8 2N7002, Q9 2N7002, U1 GW1NR-LV9-QN88-C6/I5, U10 LM393, U2 ESD224DQA, U3 MIC5203-3.3BM5, U4 APS6404L-3SQR-ZR, U5 MIC5504-1.2YM5, U6 AP62150Z6, U7 W25Q16JVUXIQ, U8 4066, U9 ESD224DQA, X1 27MHz

Commit message: Whops, failed to save schematic before commit.
Parts:
- removed D21: PESD5V0L1BSLAZ, UNIC:D_SOD-882, symbol Diode:ESD9B5.0ST5G
- removed U10: LM393, Package_SON:WSON-8-1EP_2x2mm_P0.5mm_EP0.9x1.6mm, symbol UNIC:LM393
- removed U8: 4066, Package_DFN_QFN:DHVQFN-14-1EP_2.5x3mm_P0.5mm_EP1x1.5mm, symbol 4xxx:4066
- removed U9: ESD224DQA, Package_DFN_QFN:Diodes_UDFN-10_1.0x2.5mm_P0.5mm, symbol Power_Protection:ESD224DQA
- added C24, C25, C26: 27p, UNIC:C_0402_1005Metric_Pad0.74x0.62mm_HandSolder, symbol Device:C_Small
- added C27, C28, C29, C30, C31, C32, C33, C34: 2.2u, UNIC:C_0402_1005Metric_Pad0.74x0.62mm_HandSolder, symbol Device:C_Small
- added R21: 12k, UNIC:R_0402_1005Metric_Pad0.72x0.64mm_HandSolder, symbol Device:R_Small_US
- added U11: FT232H, Package_DFN_QFN:QFN-48-1EP_8x8mm_P0.5mm_EP6.2x6.2mm, symbol Interface_USB:FT232H
- added Y1: 12MHz, symbol Device:Crystal
- J_DISPLAY1: footprint UNIC:CF31121D0R0-05-NH -> UNIC:CF4212FH0R0-05-NH
- R22: value 10k -> 12k; mpn CR0402-FX-1002GLF -> (none)
- R23: value 68.k -> 0
- R24: value 5.1k -> 0
Connections:
- net +3V3: now also R22.2, R24.2, C27.1, C28.1, C29.1, C30.1, C31.1, C32.1, U11.12 (VCCIO), U11.24 (VCCIO), U11.39 (VCCD), U11.40 (VREGIN), U11.46 (VCCIO); no longer R22.1
- net DONE: now also U11.19 (ADBUS6)
- net GND: now also C24.2, C25.2, C26.2, C27.2, C28.2, C29.2, C30.2, C31.2, C32.2, C33.2, C34.2, R21.1, U11.10 (GND), U11.11 (GND), U11.22 (GND), U11.23 (GND), U11.35 (GND), U11.36 (GND), U11.4 (AGND), U11.41 (AGND), U11.47 (GND), U11.48 (GND), U11.9 (AGND); no longer R24.1
- net JTAG_SEL_N: now also U11.17 (ADBUS4)
- net JTAG_TCK: now also U11.13 (ADBUS0)
- net JTAG_TDI: now also U11.14 (ADBUS1)
- net JTAG_TDO: now also U11.15 (ADBUS2)
- net JTAG_TMS: now also U11.16 (ADBUS3)
- net RECONFIG_N: now also U11.18 (ADBUS5)
- net USB_CC2: no longer U2.1
- net USB_DM: now also U11.6 (DM)
- net USB_DP: now also U2.1, U11.7 (DP)
- net VBUS: now also U2.4, U2.5
- net at R23.1: now also U11.3 (VPHY); no longer R24.2
- removed net USB_RXM: J1.A10 (RX2-), J1.B10 (RX1-), U2.4
- removed net USB_RXP: J1.A11 (RX2+), J1.B11 (RX1+), U2.5
- net USB_TXM: no longer names the net of J1.A3 (TX1-)
- net USB_TXM: no longer J1.B3 (TX2-)
- net USB_TXP: no longer names the net of J1.A2 (TX1+)
- net USB_TXP: no longer J1.B2 (TX2+)
- new net: C25.1, U11.2 (XCSO), Y1.2
- new net: C24.1, U11.1 (XCSI), Y1.1
- new net: C26.1, R22.1, U11.34 (~{RESET})
- new net: C34.1, U11.37 (VCCA)
- new net: C33.1, U11.38 (VCCCORE)
- new net: R21.2, U11.5 (REF)
- new net: R24.1, U11.8 (VPLL)
- no-connect marks 10 -> 28
Other:
- note added: "There are better connectors, where the appropriate pins are pre-combined making PCB design easier. Need some checking for availability."
- note removed: "Follwing the lead of: https://github.com/minoseigenheer/SWD-over-USB-C"

Commit message: Integrated JTAG controller mostly routed.
There are still some keepout violations and power nets
are incomplete, but at least there's a light at the end
if the tunnel.
Parts:
- removed C32: 2.2u, UNIC:C_0402_1005Metric_Pad0.74x0.62mm_HandSolder, symbol Device:C_Small
- C1: footprint UNIC:C_0402_1005Metric_Pad0.74x0.62mm_HandSolder -> Capacitor_SMD:C_0402_1005Metric_Pad0.74x0.62mm_HandSolder
- C10, C11, C12, C13, C14, C15, C16, C17, C18, C19, C2, C20, C21, C22, C23, C24, C25, C26, C27, C28, C29, C3, C30, C31, C33, C34, C4, C6, C9: footprint UNIC:C_0402_1005Metric_Pad0.74x0.62mm_HandSolder -> Capacitor_SMD:C_0201_0603Metric
- R1, R10, R11, R12, R13, R14, R15, R16, R17, R18, R19, R2, R20, R21, R22, R23, R24, R3, R4, R5, R6, R7, R8, R9: footprint UNIC:R_0402_1005Metric_Pad0.72x0.64mm_HandSolder -> Resistor_SMD:R_0201_0603Metric
- U11: footprint Package_DFN_QFN:QFN-48-1EP_8x8mm_P0.5mm_EP6.2x6.2mm -> Package_QFP:LQFP-48_7x7mm_P0.5mm
- Y1: footprint (none) -> Crystal:Crystal_SMD_2016-4Pin_2.0x1.6mm; symbol Device:Crystal -> Device:Crystal_GND24; mpn (none) -> E9X250101G03
Connections:
- net DONE: no longer U11.19 (ADBUS6)
- net GND: now also Y1.2, Y1.4
- net JTAG_SEL_N: no longer J_EXT1.1 (Pin_1)
- net JTAG_TCK: no longer J_EXT1.6 (Pin_6)
- net JTAG_TDI: no longer J_EXT1.2 (Pin_2)
- net JTAG_TDO: no longer J_EXT1.4 (Pin_4)
- net JTAG_TMS: no longer J_EXT1.5 (Pin_5)
- net RECONFIG_N: no longer J_EXT1.3 (Pin_3), U11.18 (ADBUS5)
- net USB_DM: now also U2.9
- net USB_DP: now also U2.10
- net at C25.1, U11.2 (XCSO): now also Y1.3; no longer Y1.2
- no-connect marks 28 -> 34

Commit message: UnIC with FT232H is fully routed.
Not all that nicely, power needs a lot more work. But at least
connectivity is there.
Parts:
- added C32: 33p, Capacitor_SMD:C_0201_0603Metric, symbol Device:C_Small
- added R25: 0, Resistor_SMD:R_0201_0603Metric, symbol Device:R_Small_US
- U6: value AP62150Z6 -> TPS562242; manufacturer Diodes Incorporated -> Texas Instruments; mpn AP62150Z6-7 -> TPS562242
- Y1: footprint Crystal:Crystal_SMD_2016-4Pin_2.0x1.6mm -> UNIC:Crystal_SMD_2016-4Pin_2.0x1.6mm
Connections:
- net +3V3: now also C32.1
- net GND: now also R25.1; no longer J1.S1 (SHIELD)
- net JTAG_SEL_N: now also U11.18 (ADBUS5); no longer U11.17 (ADBUS4)
- net SPI_IO2: no longer J_DISPLAY1.6 (Pin_6)
- net SPI_IO3: now also J_DISPLAY1.6 (Pin_6)
- net at R4.2, R5.1, U6.6 (FB): now also C32.2
- new net: J1.S1 (SHIELD), R25.2
Other:
- note added: "According to AN184, default pin behavior: ADBUS0 TXD Output ADBUS1 RXD Input-PU ADBUS2 RTS# Output ADBUS3 CTS# Input-PU ADBUS4 DTR# Output ADBUS5 DSR# Input-PU ADBUS6 DCD# Input-PU ADBUS7 RI# Input-PU So TCK and TDO might toggle during enumeration, but TMS would be held high, which will keep/reset the JTAG FSM to test-logic-reset state. Thus, no isolation is needed. Furthermore JTAG_SEL_N is pull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"
- note added: "OLED is any "Ledger Nano S" 12-pin compatible display. These are cheap on AliExpress: https://www.aliexpress.us/item/3256805237655177.html"
- note removed: "Apparently one wants an "Ledger Nano S" 12-pin compatible display. These are cheap on AliExpress and have a different pinout: https://www.aliexpress.us/item/3256805237655177.html Connector should be compatible, but placement needs to be checked. Flex still needs 'loopty-loop' around. Flex starts at 1.642mm from top here, whereas it was 3mm in the old days. Flex is 20mm long here, whereas it was 2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"
- note removed: "Display: https://www.crystalfontz.com/product/cfal12832c0091bw-small-oled-white-monochrome Other interesting displays: https://www.crystalfontz.com/product/cfaf80160a00096tn-80x160-small-color-tft-display https://www.crystalfontz.com/products/document/4618/CFAL64128B00096BWC_Datasheet.pdf"
- note removed: "ECO: change part to TPS562242"
- note removed: "There are better connectors, where the appropriate pins are pre-combined making PCB design easier. Need some checking for availability."
- moved on the sheet: C1, C10, C11, C12, C13, C14, C15, C16, C17, C18, C19, C2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

Commit message: UnIC wuth ISB (V2.0) is pretty much complete.
Other:
- note added: "Clock considerations: - 2 PLLs with a secondary output divider each, only integer mode - PLL VCO is between 400 and 1000MHz for fast, 350 to 800 for slow devices - Internal clock is 105/125MHz (based on device) - There are CLKDIV resources that support 2/3.5/4/5/(8) divisor settings"
- note added: "Issues reported with GoWin FPGAs: https://github.com/juj/gowin_flipflop_drainer Have not seen this issue, probably fixed in recent stepping"
- note added: "TODO: - Add more vias to EPAD, make sure they are of the 'ENCROACHED' style, which is to say, that they are open on the top and solder-mask-defined on the bottom. See Microchip AN18.15 for details. They recommend: 0.25-0.3mm FHS and 0.055-0.075mm larger solder mask opening. ... I don't think KiCAD can do this kind of thing."
- note removed: "Clock considerations: - 2 PLLs with a secondary output divider each, only integer mode - PLL VCO is between 400 and 1000MHz for fast, 350 to 800 for slow devices - Internal clock is based on 105/125MHz (based on device) - There are CLKDIV resources that support 2/3.5/4/5/(8) divisor settings"
- note removed: "Issues reported with GoWin FPGAs: https://github.com/juj/gowin_flipflop_drainer"
- note removed: "TODO: - Add more vias to EPAD, make sure they are of the 'ENCROACHED' style, which is to say, that they are open on the top and solder-mask-defined on the bottom. See Microchip AN18.15 for details. They recommend: 0.25-0.3mm FHS and 0.055-0.075mm larger solder mask opening. ... I don't think KiCAD can do this kind of thing. - Can we relax manufacturing cost? by making the holes 0.3mm FHS?"
- note removed: "Volume PCB Assembly BOM Total ======== ======= ========= ======= ======= 100 1.5 4.3 22.05 27.85 200 1.08 2.8 21.61 25.49 1000 0.43 1.3 19.49 21.22"
Changed lines of the file:
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@@
 	(title_block
 		(title "UNIC 40")
-		(date "2023-11-24")
-		(rev "1.0")
+		(date "2025-01-13")
+		(rev "2.0")
 		(company "Modular Circuits")
 	)
@@
 		)
 	)
-	(text "Issues reported with GoWin FPGAs:\n\nhttps://github.com/juj/gowin_flipflop_drainer"
+	(text "Issues reported with GoWin FPGAs:\nhttps://github.com/juj/gowin_flipflop_drainer\nHave not seen this issue, probably fixed in recent stepping"
 		(exclude_from_sim no)
-		(at 355.6 412.75 0)
+		(at 96.52 36.83 0)
 		(effects
 			(font
@@
 		)
 	)
-	(text "TODO:\n- Add more vias to EPAD, make sure they are of the 'ENCROACHED' style,\n  which is to say, that they are open on the top and solder-mask-defined\n  on the bottom. See Microchip AN18.15 for details. They recommend:\n  0.25-0.3mm FHS and 0.055-0.075mm larger solder mask opening.\n  ... I don't think KiCAD can do this kind of thing.\n- Can we relax manufacturing cost? by making the holes 0.3mm FHS?"
+	(text "TODO:\n- Add more vias to EPAD, make sure they are of the 'ENCROACHED' style,\n  which is to say, that they are open on the top and solder-mask-defined\n  on the bottom. See Microchip AN18.15 for details. They recommend:\n  0.25-0.3mm FHS and 0.055-0.075mm larger solder mask opening.\n  ... I don't think KiCAD can do this kind of thing."
 		(exclude_from_sim no)
-		(at 251.46 -33.02 0)
+		(at 236.22 130.81 0)
 		(effects
 			(font
@@
 		)
 	)
-	(text "Volume      PCB      Assembly   BOM      Total\n========   =======  =========  =======  =======\n100          1.5     4.3        22.05     27.85\n200          1.08    2.8        21.61     25.49\n1000         0.43    1.3        19.49     21.22"
-		(exclude_from_sim no)
-		(at 36.83 -5.08 0)
-		(effects
-			(font
-				(face "LM Mono 10")
-				(size 1.27 1.27)
-			)
-			(justify left bottom)
-		)
-	)
 	(text "VSS"
 		(exclude_from_sim no)
@@
 		)
 	)
-	(text "Clock considerations:\n- 2 PLLs with a secondary output divider each, only integer mode\n- PLL VCO is between 400 and 1000MHz for fast, 350 to 800 for slow devices\n- Internal clock is based on 105/125MHz (based on device)\n- There are CLKDIV resources that support 2/3.5/4/5/(8) divisor settings"
+	(text "Clock considerations:\n- 2 PLLs with a secondary output divider each, only integer mode\n- PLL VCO is between 400 and 1000MHz for fast, 350 to 800 for slow devices\n- Internal clock is 105/125MHz (based on device)\n- There are CLKDIV resources that support 2/3.5/4/5/(8) divisor settings"
 		(exclude_from_sim no)
-		(at 135.89 -20.32 0)
+		(at 237.49 147.32 0)
 		(effects
 			(font
@@
 	(text "QN88 package is common between N4, N9, NR4 and NR9.\nN2 also supports this package, but very different pinout\n\nCarried by RuTronic, Mouser and these guys:\nhttps://www.edgeelectronics.com/fpga/?start=49\n"
 		(exclude_from_sim no)
-		(at 109.22 27.94 0)
+		(at 96.52 27.94 0)
 		(effects
 			(font
